Commit message: fixed scaling of the robot model

File: neato_node/urdf/neato.urdf.xacro (robot description, xacro)
@@ -1,16 +1,17 @@
 <?xml version="1.0"?>
-<robot xmlns:xacro="http://ros.org/wiki/xacro" name="botsy">
+<robot xmlns:xacro="http://ros.org/wiki/xacro" name="neato">
     <link name="base_link">
       <inertial>
-        <mass value="1.477" />
+        <mass value="4.1" />
         <origin xyz="0 0 0" />
         <inertia ixx="0.01152" ixy="0.0" ixz="0.0" iyy="0.01152" iyz="0.0" izz="0.0218" />
       </inertial>
       <visual>
-        <origin xyz="0 0 0" rpy="0 0 0" />
+        <origin xyz="0 0 0" rpy="0 0 90" />
         <geometry>
-          <mesh filename="package://neato_node/meshes/neato.dae"/>
+          <mesh filename="package://neato_node/meshes/neato.dae" scale="0.01 0.01 0.01"/>
         </geometry>
       </visual>
+<!--  stl exported from sketchup broken
       <collision>
         <origin xyz="0 0 0" rpy="0 0 0" />
@@ -19,4 +20,5 @@
         </geometry>
       </collision>
+ -->
     </link>
 </robot>

Commit message: changed baseframt to laser tf to static tf2 and adapted for botvac, added more navigation visualisation to rviz, further botvacization, each neato should get its own driver class in future

File: neato_node/urdf/neato.urdf.xacro (robot description, xacro)
@@ -8,7 +8,7 @@
       </inertial>
       <visual>
-        <origin xyz="0 0 0" rpy="0 0 90" />
+        <origin xyz="0 0 0" rpy="0 0 1.57" />
         <geometry>
-          <mesh filename="package://neato_node/meshes/neato.dae" scale="0.01 0.01 0.01"/>
+          <mesh filename="package://neato_node/meshes/neato.dae" scale="0.025 0.025 0.025"/>
         </geometry>
       </visual>

Commit message: Update neato.urdf.xacro

File: neato_node/urdf/neato.urdf.xacro (robot description, xacro)
@@ -8,5 +8,5 @@
       </inertial>
       <visual>
-        <origin xyz="0 0 0" rpy="0 0 1.57" />
+        <origin xyz="0 0.25 0" rpy="0 0 1.57" />
         <geometry>
           <mesh filename="package://neato_node/meshes/neato.dae" scale="0.025 0.025 0.025"/>

Commit message: Update neato.urdf.xacro

File: neato_node/urdf/neato.urdf.xacro (robot description, xacro)
@@ -8,5 +8,5 @@
       </inertial>
       <visual>
-        <origin xyz="0 0.25 0" rpy="0 0 1.57" />
+        <origin xyz="0 -0.1 0" rpy="0 0 1.57" />
         <geometry>
           <mesh filename="package://neato_node/meshes/neato.dae" scale="0.025 0.025 0.025"/>

Commit message: Update neato.urdf.xacro

File: neato_node/urdf/neato.urdf.xacro (robot description, xacro)
@@ -8,5 +8,5 @@
       </inertial>
       <visual>
-        <origin xyz="0 -0.1 0" rpy="0 0 1.57" />
+        <origin xyz="0 -0.15 0" rpy="0 0 1.57" />
         <geometry>
           <mesh filename="package://neato_node/meshes/neato.dae" scale="0.025 0.025 0.025"/>

Commit message: Adjusted visual centre of robot model

File: neato_node/urdf/neato.urdf.xacro (robot description, xacro)
@@ -8,5 +8,5 @@
       </inertial>
       <visual>
-        <origin xyz="0 -0.15 0" rpy="0 0 1.57" />
+        <origin xyz="0.17 -0.17 0" rpy="0 0 1.57" />
         <geometry>
           <mesh filename="package://neato_node/meshes/neato.dae" scale="0.025 0.025 0.025"/>
